File: hw/bldc_driver/bldc_driver.kicad_pcb (KiCad board)
At the start: 4 copper layers, 101 x 48 mm, 150 parts, among them J1 430450412, J2 B4B-EH-A(LF)(SN), J3 B4B-EH-A(LF)(SN), J4 1733583, Q2 IRF540N, Q3 IRF540N, Q4 IRF540N, Q5 IRF540N, Q6 IRF540N, Q7 IRF540N, SW1 BTSA-N-P-1, U1 CH32V30xRxTx, U10 TPS54202DDC, U11 AMC1200BDWV, U12 AMC1200BDWV, U13 AMC1200BDWV, U14 SN65HVD230, U2 STGAP2SCM, U3 STGAP2SCM, U4 STGAP2SCM, U5 STGAP2SCM, U6 STGAP2SCM, U7 STGAP2SCM, U8 TPS54202DDC, U9 AMC1200BDWV, Y1 Crystal_GND24

Commit message: before reroute
Parts:
- removed C1, C2, C3, C4: 0.1 µF, Capacitor_SMD:C_0805_2012Metric_Pad1.18x1.45mm_HandSolder
- removed U1: CH32V30xRxTx, Package_QFP:LQFP-64_10x10mm_P0.5mm
- added C55: 10 µF, Capacitor_SMD:C_0805_2012Metric_Pad1.18x1.45mm_HandSolder, B.Cu at (157.0, 95.2)
- added C56: 0.1 µF, Capacitor_SMD:C_0805_2012Metric_Pad1.18x1.45mm_HandSolder, F.Cu at (157.1, 95.2)
- added C57: 0.1 µF, Capacitor_SMD:C_0805_2012Metric_Pad1.18x1.45mm_HandSolder, F.Cu at (156.9, 84.5)
- added C58: 0.1 µF, Capacitor_SMD:C_0805_2012Metric_Pad1.18x1.45mm_HandSolder, F.Cu at (143.7, 84.1)
- added C59: 1 µF, Capacitor_SMD:C_0805_2012Metric_Pad1.18x1.45mm_HandSolder, F.Cu at (143.0, 92.7)
- added C60: 0.1 µF, Capacitor_SMD:C_0805_2012Metric_Pad1.18x1.45mm_HandSolder, F.Cu at (146.1, 84.1)
- added C61: 10 nF, Capacitor_SMD:C_0805_2012Metric_Pad1.18x1.45mm_HandSolder, F.Cu at (145.0, 92.7)
- added R41: 0 ohm, Resistor_SMD:R_0603_1608Metric_Pad0.98x0.95mm_HandSolder, F.Cu at (159.2, 89.3)
- added R42: 0 ohm, Resistor_SMD:R_0603_1608Metric_Pad0.98x0.95mm_HandSolder, F.Cu at (159.2, 87.8)
- added R43: 0 ohm, Resistor_SMD:R_0603_1608Metric_Pad0.98x0.95mm_HandSolder, F.Cu at (157.0, 74.7)
- added R44: 0 ohm, Resistor_SMD:R_0603_1608Metric_Pad0.98x0.95mm_HandSolder, F.Cu at (155.4, 74.7)
- added U15: STM32L431CCTx, Package_QFP:LQFP-48_7x7mm_P0.5mm, F.Cu at (151.8, 90.2)
- added U16: SN74LVC1G125DBV, Package_TO_SOT_SMD:SOT-23-5_HandSoldering, B.Cu at (154.6, 99.8)
- added U17: SN74LVC1G125DBV, Package_TO_SOT_SMD:SOT-23-5_HandSoldering, B.Cu at (150.9, 99.7)
- C39: moved to B.Cu
- J2: value B4B-EH-A(LF)(SN) -> B6B-EH-A(LF)(SN); footprint Connector_JST:JST_EH_B4B-EH-A_1x04_P2.50mm_Vertical -> Connector_JST:JST_EH_B6B-EH-A_1x06_P2.50mm_Vertical
- R4: footprint Resistor_SMD:R_0201_0603Metric_Pad0.64x0.40mm_HandSolder -> Resistor_SMD:R_0603_1608Metric_Pad0.98x0.95mm_HandSolder; moved to B.Cu
- moved U3 27.8 mm to (133.0, 104.9)
- moved U7 27.8 mm to (133.0, 77.1)
- moved C43 27.6 mm to (139.9, 106.3)
- moved C52 27.6 mm to (139.8, 78.7)
- moved C44 27.4 mm to (139.8, 104.0)
- moved C51 27.4 mm to (139.8, 76.6)
- moved R33 24.9 mm to (105.1, 75.0)
- moved R35 24.9 mm to (105.1, 75.0)
- moved D10 24.8 mm to (105.0, 103.6)
- moved D13 24.8 mm to (105.1, 78.8)
- moved D14 24.8 mm to (105.1, 78.8)
- moved D9 24.8 mm to (105.0, 103.6)
- moved R12 24.8 mm to (105.0, 99.8)
- moved R27 24.8 mm to (105.0, 99.8)
- moved R13 24.7 mm to (105.0, 107.4)
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Connections:
- net /Motor/PH_U_HI renamed /PH_U_HI
- net /Motor/PH_U_LO renamed /PH_U_LO
- net /Motor/PH_V_HI renamed /PH_V_HI
- net /Motor/PH_V_LO renamed /PH_V_LO
- net /Motor/PH_W_HI renamed /PH_W_HI
- net /Motor/PH_W_LO renamed /PH_W_LO
- net Net-(U1-~{RST}) renamed /NRESET
- C41 pad 1: Net-(U1-OSC_IN) -> GND
- C41 pad 2: GND -> Net-(U15-PH0)
- C42 pad 1: Net-(U1-OSC_OUT) -> GND
- C42 pad 2: GND -> Net-(U15-PH1)
- J2 pad 2: /SWCLK -> Net-(J2-Pin_2)
- J2 pad 3: /SWDIO -> /SWCLK
- J2 pad 4: +3V3 -> /SWDIO
- J3 pad 2: /USART3_RX -> /USART1_RX
- J3 pad 3: /USART3_TX -> /USART1_TX
- TP7 pad 1: /Motor/MOTOR_W -> /Motor/MOTOR_U
- TP9 pad 1: /Motor/MOTOR_U -> /Motor/MOTOR_W
- U11 pad 6: /Motor/V_ADC_N -> /V_ADC_N
- U11 pad 7: /Motor/V_ADC_P -> /V_ADC_P
- U12 pad 6: /Motor/U_ADC_N -> /U_ADC_N
- U12 pad 7: /Motor/U_ADC_P -> /U_ADC_P
- U13 pad 6: /Motor/W_ADC_N -> /W_ADC_N
- U13 pad 7: /Motor/W_ADC_P -> /W_ADC_P
- U14 pad 1: /CAN_TX -> /CAN_RX
- U14 pad 4: /CAN_RX -> /CAN_TX
- U9 pad 6: /Motor/SHUNT_CURR_N -> /SHUNT_CURR_N
- U9 pad 7: /Motor/SHUNT_CURR_P -> /SHUNT_CURR_P
- Y1 pad 1: Net-(U1-OSC_OUT) -> Net-(U15-PH1)
- Y1 pad 3: Net-(U1-OSC_IN) -> Net-(U15-PH0)
Routing:
- net Net-(U1-OSC_OUT): track 2.42 -> 0.00 mm
- net Net-(U1-OSC_IN): track 2.40 -> 0.00 mm
Other:
- board text added: "Daniel P. & JLPF"
- board text removed: "Daniel P. (steewBSD)"
